Commit message: Colab ML pipeline, all-programme data tooling, ROS2 deployment, Qwen3 LLM
- notebooks/01-05: staged Colab A100 pipeline (clean, EDA, embeddings,
  crash-safe training, evaluation); legacy per-topic notebooks removed
- LLM: Qwen3-4B-Instruct-2507 + all-linear LoRA; HF transformers serving
  backend (LLM_BACKEND); reranker bge-reranker-v2-m3
- Data tooling (scripts): fetch_lms (c4mpus LMS sync + PDF extraction),
  fetch_softwarica_courses (official course API: fees/careers/modules),
  fetch_curriculum, import_public_postings, scrape_nepali_jobs (MeroJob +
  KumariJob real postings), export_policies (ONNX/TorchScript)
- Multi-programme: CurriculumModule.programme + content fields; parser +
  ingest content-chunking; programme-aware prompt + frontend selector
- ROS2: sim camera/world, gz_joint_relay, diagnostics_node, deployment ONNX tier
- Dashboard: /evaluation endpoint + real thesis-run analytics charts
- Real public data committed: 297 job postings (200 intl + 97 real Nepali),
  O*NET data cards. Authenticated LMS curriculum stays out of git (private).

Co-Authored-By: Claude Opus 4.8 <noreply@anthropic.com>

File: ros2_ws/src/drona_description/urdf/drona_humanoid.urdf.xacro (robot description, xacro)
@@ -9,4 +9,12 @@
 -->
 <robot xmlns:xacro="http://www.ros.org/wiki/xacro" name="drona_humanoid">
+  <!-- Simulation feature gates (harmless elsewhere: RViz/Isaac ignore <gazebo>).
+       use_gz_camera  : head camera sensor for gz sim (needs the sensors system
+                        in the world - drona_bringup/worlds/drona_advising.sdf).
+       use_gz_control : per-joint PID position controllers + joint-state
+                        publisher so the gz model mirrors /drona/joint_states
+                        (relayed by drona_ros gz_joint_relay). -->
+  <xacro:arg name="use_gz_camera" default="false"/>
+  <xacro:arg name="use_gz_control" default="false"/>
   <!-- ── Materials ─────────────────────────────────────────────────────────── -->
   <material name="drona_crimson"><color rgba="0.78 0.10 0.23 1.0"/></material>
@@ -178,3 +186,71 @@
     <limit lower="0.0" upper="1.0" effort="3" velocity="1.0"/>
   </joint>
+  <!-- ── Head camera (perception sensor) ──────────────────────────────────────
+       The physical deployment uses a webcam at eye level; this frame is its
+       TF anchor in every mode, and in Gazebo it also carries the simulated
+       camera sensor. camera_optical_frame follows REP-103 (z forward). -->
+  <link name="camera_link">
+    <visual>
+      <geometry><box size="0.02 0.05 0.02"/></geometry>
+      <material name="drona_slate"/>
+    </visual>
+    <collision><geometry><box size="0.02 0.05 0.02"/></geometry></collision>
+    <xacro:box_inertial mass="0.02"/>
+  </link>
+  <joint name="camera_fixed" type="fixed">
+    <parent link="head_link"/>
+    <child link="camera_link"/>
+    <origin xyz="0.085 0 0.02"/>
+  </joint>
+  <link name="camera_optical_frame"/>
+  <joint name="camera_optical_fixed" type="fixed">
+    <parent link="camera_link"/>
+    <child link="camera_optical_frame"/>
+    <origin xyz="0 0 0" rpy="${-pi/2} 0 ${-pi/2}"/>
+  </joint>
+  <!-- ── Gazebo camera sensor (sim only) ────────────────────────────────────── -->
+  <xacro:if value="$(arg use_gz_camera)">
+    <gazebo reference="camera_link">
+      <sensor name="drona_head_camera" type="camera">
+        <topic>drona/camera/image_raw</topic>
+        <update_rate>15</update_rate>
+        <always_on>1</always_on>
+        <visualize>true</visualize>
+        <gz_frame_id>camera_optical_frame</gz_frame_id>
+        <camera>
+          <horizontal_fov>1.204</horizontal_fov>
+          <image><width>640</width><height>480</height><format>R8G8B8</format></image>
+          <clip><near>0.05</near><far>10.0</far></clip>
+          <camera_info_topic>drona/camera/camera_info</camera_info_topic>
+        </camera>
+      </sensor>
+    </gazebo>
+  </xacro:if>
+  <!-- ── Gazebo joint control (sim only) ──────────────────────────────────────
+       PID position controllers per joint; the drona_ros gz_joint_relay node
+       converts /drona/joint_states into these per-joint command topics (bridged
+       to gz.msgs.Double), so the gz model performs the same gestures as the
+       policy publishes - the sim mirrors deployment exactly. -->
+  <xacro:if value="$(arg use_gz_control)">
+    <gazebo>
+      <plugin filename="gz-sim-joint-state-publisher-system"
+              name="gz::sim::systems::JointStatePublisher"/>
+      <xacro:macro name="gz_joint_pid" params="joint">
+        <plugin filename="gz-sim-joint-position-controller-system"
+                name="gz::sim::systems::JointPositionController">
+          <joint_name>${joint}</joint_name>
+          <topic>drona/gz/${joint}_cmd</topic>
+          <p_gain>20.0</p_gain>
+          <i_gain>0.5</i_gain>
+          <d_gain>1.0</d_gain>
+        </plugin>
+      </xacro:macro>
+      <xacro:gz_joint_pid joint="j0_base_yaw"/>
+      <xacro:gz_joint_pid joint="j1_shoulder"/>
+      <xacro:gz_joint_pid joint="j2_elbow"/>
+      <xacro:gz_joint_pid joint="j3_wrist_pitch"/>
+      <xacro:gz_joint_pid joint="j4_wrist_roll"/>
+      <xacro:gz_joint_pid joint="j5_gripper"/>
+    </gazebo>
+  </xacro:if>
 </robot>

Commit message: sim: restyle the robot and build a college advising room
THE ROBOT
---------
The arm segments were coloured green / red / yellow / blue - useful debug
colouring for spotting a mis-parented joint, but it reads as a toy - and the head
was a flesh-toned sphere with no front, so you could not tell which way the robot
was facing. For a robot whose whole behaviour is approach-and-greet, orientation
has to be readable at a glance.

Rebuilt around one palette (light shell, graphite joints, crimson accent) with a
dark visor and two emissive eyes giving a clear front, a chest display, tapered
torso, joint caps on the arm, a two-finger hand, a rounded base skirt with a
bumper ring and a forward sensor strip, and hub caps so a rolling wheel visibly
rolls.

Done entirely with multiple <visual> blocks per link, which URDF allows. No new
links, so the TF tree, joint_states and the controllers cannot be affected -
verified by generating the URDF before and after and diffing: joints identical,
collisions identical, visual blocks 14 -> 33. Both use_mobile_base modes parse.

No meshes are downloaded, so the sim still starts offline and the repo gains no
binary assets.

THE ROOM
--------
A bare ground plane made the sim read as a physics test rather than a place a
student walks into. drona_advising.sdf now contains a Softwarica advising room:
floor slab, four walls with an open doorway side, whiteboard, crimson notice
board, banner, two rows of student desks with chairs, a waiting bench, a
bookshelf and greenery - 68 models, all static primitives.

Added three point lights: the single directional "sun" lights an outdoor scene
and left the interior a dark box.

The robot, the advising desk and the student figure keep their original poses, so
perception framing and the approach behaviour are unchanged. `gz sdf -k` reports
Valid.

DOCS
----
docs/INTERACTING_WITH_DRONA.md answers "how do I interact and how does it speak":
the interaction loop, the three ways in (web console, ros2 topic pub, walking the
student figure up to it in Gazebo), and the speech backends.

Verified state of audio on this machine, which is not obvious: WSL2 has no
/dev/snd sound card, but WSLg exposes a PulseAudio socket and PULSE_SERVER is
already set, so sound does reach the Windows speakers. What is missing is the
software - espeak-ng, ffplay, aplay and paplay are all absent, so the robot
currently cannot speak. `sudo apt install -y espeak-ng pulseaudio-utils` fixes it.
speech_node already degrades to the log backend when espeak is missing, so the
sim launches cleanly meanwhile and prints what it would have said.

497 python tests pass.

Co-Authored-By: Claude Opus 4.8 <noreply@anthropic.com>

File: ros2_ws/src/drona_description/urdf/drona_humanoid.urdf.xacro (robot description, xacro)
@@ -24,11 +24,22 @@
   <xacro:arg name="use_mobile_base" default="false"/>
   <!-- ── Materials ─────────────────────────────────────────────────────────── -->
-  <material name="drona_crimson"><color rgba="0.78 0.10 0.23 1.0"/></material>
-  <material name="drona_slate"><color rgba="0.25 0.28 0.34 1.0"/></material>
-  <material name="drona_green"><color rgba="0.30 0.80 0.30 1.0"/></material>
-  <material name="drona_red"><color rgba="0.80 0.30 0.30 1.0"/></material>
-  <material name="drona_yellow"><color rgba="0.85 0.80 0.30 1.0"/></material>
-  <material name="drona_blue"><color rgba="0.35 0.45 0.90 1.0"/></material>
-  <material name="drona_skin"><color rgba="0.90 0.78 0.68 1.0"/></material>
+  <!-- Palette. The previous per-link rainbow (green upper arm, red forearm,
+       yellow wrist) was debug colouring: useful for spotting a mis-parented
+       joint, but it reads as a toy. A service robot that students are meant to
+       approach needs a coherent product palette - a light shell, dark structural
+       joints, one accent colour, and an emissive face. -->
+  <material name="drona_shell">   <color rgba="0.94 0.94 0.96 1.0"/></material>
+  <material name="drona_graphite"><color rgba="0.16 0.17 0.20 1.0"/></material>
+  <material name="drona_slate">   <color rgba="0.31 0.34 0.40 1.0"/></material>
+  <material name="drona_crimson"> <color rgba="0.78 0.10 0.23 1.0"/></material>
+  <material name="drona_screen">  <color rgba="0.05 0.06 0.09 1.0"/></material>
+  <material name="drona_eye">     <color rgba="0.20 0.85 0.95 1.0"/></material>
+  <material name="drona_rubber">  <color rgba="0.10 0.10 0.12 1.0"/></material>
+  <!-- Kept so any external xacro referencing the old names still resolves. -->
+  <material name="drona_green">   <color rgba="0.94 0.94 0.96 1.0"/></material>
+  <material name="drona_red">     <color rgba="0.94 0.94 0.96 1.0"/></material>
+  <material name="drona_yellow">  <color rgba="0.31 0.34 0.40 1.0"/></material>
+  <material name="drona_blue">    <color rgba="0.31 0.34 0.40 1.0"/></material>
+  <material name="drona_skin">    <color rgba="0.94 0.94 0.96 1.0"/></material>
   <!-- Reusable inertial macro (small solid-ish box approximation). -->
   <xacro:macro name="box_inertial" params="mass">
@@ -41,8 +52,31 @@
   <!-- ── Torso (root) ──────────────────────────────────────────────────────── -->
   <link name="base_link">
+    <!-- Multiple <visual> blocks compose the form. URDF allows this, and it
+         adds detail without adding links, so the TF tree, joint_states and the
+         controllers are all untouched. Collision stays a single cheap box. -->
     <visual>
       <origin xyz="0 0 0.20"/>
-      <geometry><box size="0.22 0.14 0.40"/></geometry>
-      <material name="drona_slate"/>
+      <geometry><cylinder radius="0.115" length="0.34"/></geometry>
+      <material name="drona_shell"/>
+    </visual>
+    <visual>  <!-- shoulder yoke -->
+      <origin xyz="0 0 0.375"/>
+      <geometry><cylinder radius="0.105" length="0.05"/></geometry>
+      <material name="drona_graphite"/>
+    </visual>
+    <visual>  <!-- waist taper into the base -->
+      <origin xyz="0 0 0.025"/>
+      <geometry><cylinder radius="0.095" length="0.05"/></geometry>
+      <material name="drona_graphite"/>
+    </visual>
+    <visual>  <!-- chest display: what a student reads at eye-in height -->
+      <origin xyz="0.10 0 0.24"/>
+      <geometry><box size="0.02 0.15 0.11"/></geometry>
+      <material name="drona_screen"/>
+    </visual>
+    <visual>  <!-- accent band -->
+      <origin xyz="0 0 0.12"/>
+      <geometry><cylinder radius="0.117" length="0.02"/></geometry>
+      <material name="drona_crimson"/>
     </visual>
     <collision>
@@ -54,7 +88,28 @@
   <!-- Head (fixed) -->
   <link name="head_link">
-    <visual>
-      <geometry><sphere radius="0.09"/></geometry>
-      <material name="drona_skin"/>
+    <visual>  <!-- cranial shell -->
+      <geometry><sphere radius="0.095"/></geometry>
+      <material name="drona_shell"/>
+    </visual>
+    <visual>  <!-- dark visor: gives the head a clear FRONT, so a student can
+                   tell at a glance whether the robot is facing them -->
+      <origin xyz="0.055 0 0.01" rpy="0 0.25 0"/>
+      <geometry><box size="0.055 0.13 0.085"/></geometry>
+      <material name="drona_screen"/>
+    </visual>
+    <visual>  <!-- eyes: emissive-looking, the main cue that it is awake -->
+      <origin xyz="0.082 0.035 0.02" rpy="0 ${pi/2} 0"/>
+      <geometry><cylinder radius="0.016" length="0.012"/></geometry>
+      <material name="drona_eye"/>
+    </visual>
+    <visual>
+      <origin xyz="0.082 -0.035 0.02" rpy="0 ${pi/2} 0"/>
+      <geometry><cylinder radius="0.016" length="0.012"/></geometry>
+      <material name="drona_eye"/>
+    </visual>
+    <visual>  <!-- neck collar -->
+      <origin xyz="0 0 -0.075"/>
+      <geometry><cylinder radius="0.045" length="0.05"/></geometry>
+      <material name="drona_graphite"/>
     </visual>
     <collision><geometry><sphere radius="0.09"/></geometry></collision>
@@ -69,6 +124,6 @@
   <link name="arm_base">
     <visual>
-      <geometry><cylinder radius="0.04" length="0.05"/></geometry>
-      <material name="drona_crimson"/>
+      <geometry><sphere radius="0.045"/></geometry>
+      <material name="drona_graphite"/>
     </visual>
     <collision><geometry><cylinder radius="0.04" length="0.05"/></geometry></collision>
@@ -83,5 +138,9 @@
   <link name="shoulder_link">
     <visual>
-      <geometry><cylinder radius="0.035" length="0.04"/></geometry>
+      <geometry><cylinder radius="0.038" length="0.042"/></geometry>
+      <material name="drona_graphite"/>
+    </visual>
+    <visual>  <!-- crimson ring marks a driven axis -->
+      <geometry><cylinder radius="0.040" length="0.014"/></geometry>
       <material name="drona_crimson"/>
     </visual>
@@ -98,8 +157,13 @@
   <!-- ── j1: shoulder pitch ───────────────────────────────────────────────── -->
   <link name="upper_arm">
-    <visual>
-      <origin xyz="0 0 0.075"/>
-      <geometry><cylinder radius="0.025" length="0.15"/></geometry>
-      <material name="drona_green"/>
+    <visual>  <!-- upper-arm shell -->
+      <origin xyz="0 0 0.078"/>
+      <geometry><cylinder radius="0.030" length="0.13"/></geometry>
+      <material name="drona_shell"/>
+    </visual>
+    <visual>  <!-- elbow joint cap -->
+      <origin xyz="0 0 0.15"/>
+      <geometry><sphere radius="0.032"/></geometry>
+      <material name="drona_graphite"/>
     </visual>
     <collision>
@@ -118,8 +182,13 @@
   <!-- ── j2: elbow ────────────────────────────────────────────────────────── -->
   <link name="forearm">
-    <visual>
-      <origin xyz="0 0 0.06"/>
-      <geometry><cylinder radius="0.02" length="0.12"/></geometry>
-      <material name="drona_red"/>
+    <visual>  <!-- forearm shell -->
+      <origin xyz="0 0 0.058"/>
+      <geometry><cylinder radius="0.026" length="0.10"/></geometry>
+      <material name="drona_shell"/>
+    </visual>
+    <visual>  <!-- wrist joint cap -->
+      <origin xyz="0 0 0.12"/>
+      <geometry><sphere radius="0.027"/></geometry>
+      <material name="drona_graphite"/>
     </visual>
     <collision>
@@ -139,7 +208,7 @@
   <link name="wrist_pitch_link">
     <visual>
-      <origin xyz="0 0 0.035"/>
-      <geometry><cylinder radius="0.015" length="0.07"/></geometry>
-      <material name="drona_yellow"/>
+      <origin xyz="0 0 0.033"/>
+      <geometry><cylinder radius="0.019" length="0.06"/></geometry>
+      <material name="drona_slate"/>
     </visual>
     <collision>
@@ -160,6 +229,6 @@
     <visual>
       <origin xyz="0 0 0.02"/>
-      <geometry><cylinder radius="0.012" length="0.04"/></geometry>
-      <material name="drona_blue"/>
+      <geometry><cylinder radius="0.017" length="0.035"/></geometry>
+      <material name="drona_graphite"/>
     </visual>
     <collision>
@@ -178,7 +247,17 @@
   <!-- ── j5: gripper (prismatic) ──────────────────────────────────────────── -->
   <link name="gripper_link">
-    <visual>
-      <geometry><box size="0.03 0.02 0.02"/></geometry>
-      <material name="drona_crimson"/>
+    <visual>  <!-- palm -->
+      <geometry><box size="0.045 0.032 0.018"/></geometry>
+      <material name="drona_shell"/>
+    </visual>
+    <visual>  <!-- two fingers read as a hand; one block reads as a stump -->
+      <origin xyz="0.018 0.011 0.022"/>
+      <geometry><box size="0.012 0.010 0.032"/></geometry>
+      <material name="drona_graphite"/>
+    </visual>
+    <visual>
+      <origin xyz="0.018 -0.011 0.022"/>
+      <geometry><box size="0.012 0.010 0.032"/></geometry>
+      <material name="drona_graphite"/>
     </visual>
     <collision><geometry><box size="0.03 0.02 0.02"/></geometry></collision>
@@ -197,7 +276,12 @@
        camera sensor. camera_optical_frame follows REP-103 (z forward). -->
   <link name="camera_link">
-    <visual>
-      <geometry><box size="0.02 0.05 0.02"/></geometry>
-      <material name="drona_slate"/>
+    <visual>  <!-- camera housing, recessed into the visor -->
+      <geometry><box size="0.012 0.055 0.016"/></geometry>
+      <material name="drona_graphite"/>
+    </visual>
+    <visual>  <!-- lens -->
+      <origin xyz="0.008 0 0" rpy="0 ${pi/2} 0"/>
+      <geometry><cylinder radius="0.007" length="0.006"/></geometry>
+      <material name="drona_screen"/>
     </visual>
     <collision><geometry><box size="0.02 0.05 0.02"/></geometry></collision>
@@ -272,8 +356,24 @@
     <xacro:property name="chassis_h"    value="0.10"/>
     <link name="mobile_base_link">
-      <visual>
+      <visual>  <!-- rounded skirt: a cylinder reads as a service-robot base,
+                      a bare box reads as a crate -->
         <origin xyz="0 0 ${chassis_h/2}"/>
-        <geometry><box size="0.36 0.30 ${chassis_h}"/></geometry>
-        <material name="drona_base"><color rgba="0.25 0.28 0.35 1"/></material>
+        <geometry><cylinder radius="0.185" length="${chassis_h}"/></geometry>
+        <material name="drona_shell"/>
+      </visual>
+      <visual>  <!-- dark bumper ring at floor level -->
+        <origin xyz="0 0 0.022"/>
+        <geometry><cylinder radius="0.192" length="0.032"/></geometry>
+        <material name="drona_graphite"/>
+      </visual>
+      <visual>  <!-- top deck the torso sits on -->
+        <origin xyz="0 0 ${chassis_h}"/>
+        <geometry><cylinder radius="0.16" length="0.02"/></geometry>
+        <material name="drona_graphite"/>
+      </visual>
+      <visual>  <!-- forward-facing sensor strip: shows which way is 'front' -->
+        <origin xyz="0.17 0 ${chassis_h*0.7}"/>
+        <geometry><box size="0.02 0.14 0.03"/></geometry>
+        <material name="drona_screen"/>
       </visual>
       <collision>
@@ -293,6 +393,11 @@
         <visual>
           <origin rpy="1.5708 0 0"/>
-          <geometry><cylinder radius="${wheel_radius}" length="0.04"/></geometry>
-          <material name="drona_wheel"><color rgba="0.1 0.1 0.12 1"/></material>
+          <geometry><cylinder radius="${wheel_radius}" length="0.045"/></geometry>
+          <material name="drona_rubber"/>
+        </visual>
+        <visual>  <!-- hub cap, so a rolling wheel is visibly rolling -->
+          <origin rpy="1.5708 0 0"/>
+          <geometry><cylinder radius="${wheel_radius*0.45}" length="0.048"/></geometry>
+          <material name="drona_slate"/>
         </visual>
         <collision>
