Commit message: feat: Romanised Nepali routing, web voice counselling, humanoid counsellor
ROMANISED NEPALI - a real routing bug
-------------------------------------
language.py documented itself as handling code-switching, but the Devanagari
ratio test only fires when Devanagari is actually present. Nepali typed in Latin
script - "malai data science ramro lagcha, kun module ramro cha?" - scores 0.0
and was silently served by the English model. That is how most students actually
type, so this was the common case failing, not an edge case.

Added a 91-word lexicon of Romanised Nepali function words (pronouns, copulas,
postpositions, question words), curated for NON-collision with English. Content
words are excluded deliberately: they are where the two languages collide.
Firing needs two markers, or one in a short query, so a stray token in a long
English sentence cannot flip the language.

The two failure modes are not symmetric and the detector is tuned accordingly:
serving Nepali in English is bad, but serving English in Nepali is worse - a
student who asked in English and got Nepali back assumes the system is broken.
31 tests pin both directions, including adversarial English ("The cat sat on a
mat in the sun"), plus parity tests that fail if the TS and Python lexicons drift.

WEB VOICE COUNSELLING (/counsel)
--------------------------------
The robot speaks through speech_node inside WSL, which a student on their own
laptop cannot reach. /counsel runs the same loop - speak, retrieve, debias,
advise, speak back - on the browser's Web Speech API: no key, no network service,
no install. Bias flags show their verified evidence span inside the student's own
words, and pathways come back with modules and confidence.

Speech support is uneven and that is surfaced rather than hidden: recognition is
Chromium-only, and Nepali voices are often absent, so the page states what this
browser can actually do and falls back to typing. Nepali synthesis falls back
ne -> hi -> default, since Devanagari read by a Hindi voice is much closer than
an English voice attempting Nepali.

HUMANOID COUNSELLOR + STUDENT
-----------------------------
The robot had ONE arm, so it read as a manipulator on a plinth. Added a passive
left arm, hair, a blazer shoulder line, collar and a staff badge. The left arm is
deliberately passive - claiming two actuated arms would misrepresent the hardware
the thesis describes.

All of it attaches with FIXED joints and carries NO collision geometry. Verified
by regenerating the URDF: the 8 moving joints are unchanged, every original
collision is intact, and every new link has no collision - so the gesture
policies, controllers and physics are provably untouched.

The student figure was a cylinder with a ball on top. It is now recognisably a
student - shirt, jeans, shoes, hair, backpack - with the collision volume and
both link poses unchanged, so perception framing and approach behaviour are
identical. gz sdf reports Valid.

HONEST LIMIT: this is stylised, not photoreal. Photorealism needs rigged
character meshes - licensing, hundreds of MB, a network fetch - and the sim is
deliberately asset-free so it starts offline. These read clearly as a counsellor
and a student; they are not a rendered human.

20 routes build, tsc and eslint clean, 528 python tests pass.

Co-Authored-By: Claude Opus 4.8 <noreply@anthropic.com>

File: ros2_ws/src/drona_description/urdf/drona_humanoid.urdf.xacro (robot description, xacro)
@@ -36,4 +36,6 @@
   <material name="drona_eye">     <color rgba="0.20 0.85 0.95 1.0"/></material>
   <material name="drona_rubber">  <color rgba="0.10 0.10 0.12 1.0"/></material>
+  <material name="drona_hair">    <color rgba="0.09 0.07 0.07 1.0"/></material>
+  <material name="drona_attire">  <color rgba="0.16 0.26 0.42 1.0"/></material>
   <!-- Kept so any external xacro referencing the old names still resolves. -->
   <material name="drona_green">   <color rgba="0.94 0.94 0.96 1.0"/></material>
@@ -270,4 +272,130 @@
     <axis xyz="1 0 0"/>
     <limit lower="0.0" upper="1.0" effort="3" velocity="1.0"/>
+  </joint>
+  <!-- ══ Counsellor presentation: passive left arm, hair, attire ═══════════════
+       The robot had ONE arm, so it read as a manipulator on a plinth rather than
+       a person. A counselling robot a student is meant to approach and talk to
+       has to read as humanoid before it reads as a machine.
+       Every link below is attached with a FIXED joint. Fixed joints do not appear
+       in joint_states and carry no controller, so the 6-DOF actuated right arm,
+       the gesture policies and the trajectory code are all completely unaffected -
+       this is presentation only. The left arm is deliberately passive: claiming
+       two actuated arms would misrepresent the hardware the thesis describes.
+  ═══════════════════════════════════════════════════════════════════════════ -->
+  <!-- Hair: a darker mass behind and above the visor. This is the single cue
+       that most strongly reads as "a person, and a woman" at a glance, which is
+       what the counsellor framing needs. -->
+  <link name="hair_back">
+    <visual>
+      <origin xyz="-0.022 0 0.012"/>
+      <geometry><sphere radius="0.098"/></geometry>
+      <material name="drona_hair"/>
+    </visual>
+    <xacro:box_inertial mass="0.01"/>
+  </link>
+  <joint name="hair_back_fixed" type="fixed">
+    <parent link="head_link"/><child link="hair_back"/>
+    <origin xyz="0 0 0"/>
+  </joint>
+  <link name="hair_bun">
+    <visual>
+      <geometry><sphere radius="0.052"/></geometry>
+      <material name="drona_hair"/>
+    </visual>
+    <xacro:box_inertial mass="0.01"/>
+  </link>
+  <joint name="hair_bun_fixed" type="fixed">
+    <parent link="head_link"/><child link="hair_bun"/>
+    <origin xyz="-0.072 0 0.058"/>
+  </joint>
+  <!-- Shoulders / blazer line: squares off the torso into a professional
+       silhouette instead of a bare cylinder. -->
+  <link name="attire_shoulders">
+    <visual>
+      <geometry><box size="0.20 0.34 0.075"/></geometry>
+      <material name="drona_attire"/>
+    </visual>
+    <xacro:box_inertial mass="0.02"/>
+  </link>
+  <joint name="attire_shoulders_fixed" type="fixed">
+    <parent link="base_link"/><child link="attire_shoulders"/>
+    <origin xyz="0 0 0.345"/>
+  </joint>
+  <link name="attire_collar">
+    <visual>
+      <geometry><cylinder radius="0.062" length="0.05"/></geometry>
+      <material name="drona_attire"/>
+    </visual>
+    <xacro:box_inertial mass="0.01"/>
+  </link>
+  <joint name="attire_collar_fixed" type="fixed">
+    <parent link="base_link"/><child link="attire_collar"/>
+    <origin xyz="0 0 0.425"/>
+  </joint>
+  <!-- Staff badge: signals "counsellor", the way a real advisor wears one. -->
+  <link name="staff_badge">
+    <visual>
+      <geometry><box size="0.012 0.055 0.075"/></geometry>
+      <material name="drona_crimson"/>
+    </visual>
+    <xacro:box_inertial mass="0.005"/>
+  </link>
+  <joint name="staff_badge_fixed" type="fixed">
+    <parent link="base_link"/><child link="staff_badge"/>
+    <origin xyz="0.105 0.072 0.325"/>
+  </joint>
+  <!-- Passive LEFT arm, mirroring the actuated right arm's proportions so the
+       two read as a pair. Posed in a relaxed, open resting position - crossed or
+       rigid arms read as closed body language, which is wrong for counselling. -->
+  <link name="left_shoulder">
+    <visual><geometry><sphere radius="0.045"/></geometry>
+      <material name="drona_graphite"/></visual>
+    <xacro:box_inertial mass="0.05"/>
+  </link>
+  <joint name="left_shoulder_fixed" type="fixed">
+    <parent link="base_link"/><child link="left_shoulder"/>
+    <origin xyz="0 0.13 0.36"/>
+  </joint>
+  <link name="left_upper_arm">
+    <visual>
+      <origin xyz="0 0 -0.078"/>
+      <geometry><cylinder radius="0.030" length="0.13"/></geometry>
+      <material name="drona_attire"/>
+    </visual>
+    <xacro:box_inertial mass="0.05"/>
+  </link>
+  <joint name="left_upper_arm_fixed" type="fixed">
+    <parent link="left_shoulder"/><child link="left_upper_arm"/>
+    <origin xyz="0 0.012 0" rpy="-0.20 0 0"/>
+  </joint>
+  <link name="left_elbow">
+    <visual><geometry><sphere radius="0.032"/></geometry>
+      <material name="drona_graphite"/></visual>
+    <xacro:box_inertial mass="0.03"/>
+  </link>
+  <joint name="left_elbow_fixed" type="fixed">
+    <parent link="left_upper_arm"/><child link="left_elbow"/>
+    <origin xyz="0 0 -0.15"/>
+  </joint>
+  <link name="left_forearm">
+    <visual>
+      <origin xyz="0.045 0 -0.02"/>
+      <geometry><cylinder radius="0.026" length="0.10"/></geometry>
+      <material name="drona_shell"/>
+    </visual>
+    <xacro:box_inertial mass="0.04"/>
+  </link>
+  <joint name="left_forearm_fixed" type="fixed">
+    <parent link="left_elbow"/><child link="left_forearm"/>
+    <origin xyz="0 0 0" rpy="0 -1.05 0"/>
+  </joint>
+  <link name="left_hand">
+    <visual><geometry><box size="0.045 0.032 0.018"/></geometry>
+      <material name="drona_shell"/></visual>
+    <xacro:box_inertial mass="0.02"/>
+  </link>
+  <joint name="left_hand_fixed" type="fixed">
+    <parent link="left_forearm"/><child link="left_hand"/>
+    <origin xyz="0.10 0 -0.02"/>
   </joint>
   <!-- ── Head camera (perception sensor) ──────────────────────────────────────
